File: namecard.kicad_sch (KiCad schematic)
At the start: 43 parts, among them J1 Conn_01x24, J2 Conn_01x05, Q1 AO3400A, U1 STM32G030K6Tx, U2 ST25DV04K-IER8C3, U3 TPS22917DBV

Commit message: wip: 配置を更新
Parts:
- added C20: 100nf, Capacitor_SMD:C_0603_1608Metric, symbol Device:C
- added C24, C26: 0.1uf, Capacitor_SMD:C_0805_2012Metric, symbol Device:C
- added C25: 1uf, Capacitor_SMD:C_0805_2012Metric, symbol Device:C
- C23: value 22uf -> 1uf; JLCPCB C45783 -> (none)
Connections:
- net GND: now also C20.2, C24.2, C25.2, C26.2
- net SYS_VDD: now also C20.1, C25.1, C26.1
- net V_EH_RAW: now also C24.1
