File: namecard.kicad_sch (KiCad schematic)
At the start: 47 parts, among them J1 Conn_01x24, J2 Conn_01x05, Q1 AO3400A, U1 STM32G030K6Tx, U2 ST25DV04K-IER8C3, U3 TPS22917DBV

Commit message: v3向けの検証
Parts:
- U2: value ST25DV04K-IER8C3 -> ST25DV64K-IER8S3; JLCPCB C2908287 -> C1852798
Changed lines of the file:
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@@
 			)
 		)
-		(property "Value" "ST25DV04K-IER8C3"
+		(property "Value" "ST25DV64K-IER8S3"
 			(at 136.525 139.7 0)
 			(show_name no)
@@
 			)
 		)
-		(property "Datasheet" "https://www.st.com/resource/en/datasheet/st25dv04k.pdf"
+		(property "Datasheet" "https://www.st.com/resource/en/datasheet/st25dv64k.pdf"
 			(at 125.73 133.35 0)
 			(hide yes)
@@
 			)
 		)
-		(property "Description" "Dynamic NFC/RFID tag IC with 4-Kbit EEPROM, UFDFPN-8"
+		(property "Description" ""
 			(at 125.73 133.35 0)
 			(hide yes)
@@
 			)
 		)
-		(property "JLCPCB" "C2908287"
+		(property "JLCPCB" "C1852798"
 			(at 125.73 133.35 0)
 			(hide yes)

Commit message: v4
Parts:
- added C27: 1nF, Capacitor_SMD:C_0402_1005Metric, symbol Device:C
- added C28, C41, C43, C44, C45: 100nF, Capacitor_SMD:C_0402_1005Metric, symbol Device:C
- added C29, C30, C31, C32, C42: 22uF 6.3V X5R, Capacitor_SMD:C_0805_2012Metric, symbol Device:C
- added C39: 220uF/6.3V VRAW, Capacitor_Tantalum_SMD:CP_EIA-3528-21_Kemet-B, symbol Device:C
- added C40: 10uF 25V X5R, Capacitor_SMD:C_0805_2012Metric, symbol Device:C
- added C46, C48, C49: 220uF/6.3V VRES, Capacitor_Tantalum_SMD:CP_EIA-3528-21_Kemet-B, symbol Device:C
- added C47: 100nF U2 DECOUPLING, Capacitor_SMD:C_0603_1608Metric, symbol Device:C
- added D5, D6: 1N4148W, Diode_SMD:D_SOD-123, symbol Device:D
- added J3: EXT_VRES_CAP_DNP, Connector_PinHeader_2.54mm:PinHeader_1x02_P2.54mm_Vertical, symbol Connector_Generic:Conn_01x02
- added L2: 2.2uH, Inductor_SMD:L_Sunlord_SWPA252012S, symbol Device:L
- added R10: 5.11k 1% (2.5mA), Resistor_SMD:R_0402_1005Metric, symbol Device:R
- added R11: 16.2k 1%, Resistor_SMD:R_0402_1005Metric, symbol Device:R
- added R12: 0R, Resistor_SMD:R_0402_1005Metric, symbol Device:R
- added R13: 10k GPO PULLUP, Resistor_SMD:R_0603_1608Metric, symbol Device:R
- added R14: 1k EPD DISCHARGE, Resistor_SMD:R_0603_1608Metric, symbol Device:R
- added R7: 4.7M, Resistor_SMD:R_0402_1005Metric, symbol Device:R
- added R8: 1k, Resistor_SMD:R_0402_1005Metric, symbol Device:R
- added R9: 36.5k 1%, Resistor_SMD:R_0402_1005Metric, symbol Device:R
- added TP10: VRAW_TP, TestPoint:TestPoint_Pad_D1.0mm, symbol Connector:TestPoint
- added TP11: VRES_3V3_TP, TestPoint:TestPoint_Pad_D1.0mm, symbol Connector:TestPoint
- added TP12: EN_3V3_TP, TestPoint:TestPoint_Pad_D1.0mm, symbol Connector:TestPoint
- added TP8: SYS_VDD_TP, TestPoint:TestPoint_Pad_D1.0mm, symbol Connector:TestPoint
- added TP9: PWR_REQ_TP, TestPoint:TestPoint_Pad_D1.0mm, symbol Connector:TestPoint
- added U4: TPS22917DBV, Package_TO_SOT_SMD:SOT-23-6, symbol Power_Management:TPS22917DBV
- added U5: TPS3839K33DBZR, Package_TO_SOT_SMD:SOT-23, symbol Power_Supervisor:TPS3839DBZ
- added U6: LM66100, Package_TO_SOT_SMD:SOT-363_SC-70-6, symbol Power_Management:LM66100DCK
- added U7: TPS63900, Package_SON:WSON-10-1EP_2.5x2.5mm_P0.5mm_EP1.2x2mm_ThermalVias, symbol Regulator_Switching:TPS63900
- C1, C10, C11, C12, C2, C5, C6, C7, C9: value 1uF -> 1uF 50V X5R; JLCPCB (none) -> C15849; LCSC (none) -> C15849; MPN (none) -> CL10A105KB8NNNC
- C13, C18, C20, C8: JLCPCB (none) -> C14663; LCSC (none) -> C14663; MPN (none) -> CC0603KRX7R9BB104
- C14, C15, C16, C17: value 220uf -> 220uF/6.3V; footprint Capacitor_Tantalum_SMD:6TPE220MAZB -> Capacitor_Tantalum_SMD:CP_EIA-3528-21_Kemet-B; JLCPCB C79111 -> C30242; LCSC (none) -> C30242; MPN (none) -> TLJB227M006R0500
- C19: value 1nf -> 1nF; JLCPCB (none) -> C1588; LCSC (none) -> C1588; MPN (none) -> CL10B102KB8NNNC
- C23, C25: JLCPCB (none) -> C28323; LCSC (none) -> C28323; MPN (none) -> CL21B105KBFNNNE
- C24, C26: JLCPCB (none) -> C28233; LCSC (none) -> C28233; MPN (none) -> CL21B104KCFNNNE
- C3: value 4.7uF -> 4.7uF 25V X5R; footprint Capacitor_SMD:C_0603_1608Metric -> Capacitor_SMD:C_0805_2012Metric; JLCPCB (none) -> C722528; LCSC (none) -> C722528; MPN (none) -> CL21A475KAQNNNG
- C4: value 4.7uF -> 4.7uF 16V X5R; JLCPCB (none) -> C19666; LCSC (none) -> C19666; MPN (none) -> CL10A475KO8NNNC
- D1, D2, D3: value MBR0530 -> MBR0530T1G; JLCPCB (none) -> C82046; LCSC (none) -> C82046; MPN (none) -> MBR0530T1G
- D4: value D_Schottky -> DNP SCHOTTKY; DNP (none) -> 1; LCSC (none) -> C110921; MPN (none) -> PMEG2010AEH,115; now not fitted
- J1: LCSC (none) -> C506794; MPN (none) -> FH12A-24S-0.5SH(55)
- J2: JLCPCB (none) -> C5156614; LCSC (none) -> C5156614; MPN (none) -> 2.54-1*5
- L1: footprint Inductor_SMD:L_1210_3225Metric -> Inductor_SMD:L_APV_ANR4020; JLCPCB C66936 -> C6364799; LCSC (none) -> C6364799; MPN (none) -> ANR4020T470M
- Q1: JLCPCB (none) -> C20917; LCSC (none) -> C20917; MPN (none) -> AO3400A
- R1: JLCPCB (none) -> C22935; LCSC (none) -> C22935; MPN (none) -> 0603WAF1004T5E
- R2: JLCPCB (none) -> C22939; LCSC (none) -> C22939; MPN (none) -> 0603WAF220KT5E
- R3: value 1M -> 1M DNP; JLCPCB (none) -> C22935; LCSC (none) -> C22935; MPN (none) -> 0603WAF1004T5E; now not fitted
- R4, R6: JLCPCB (none) -> C25804; LCSC (none) -> C25804; MPN (none) -> 0603WAF1002T5E
- R5: value 470k -> 470k DNP; JLCPCB (none) -> C23178; LCSC (none) -> C23178; MPN (none) -> 0603WAF4703T5E; now not fitted
- TP1: value TestPoint -> VRES_3V3_TP; now left out of the parts list
- TP3: value TestPoint -> V_EH_RAW_TP; now left out of the parts list
- TP4, TP5, TP7: now left out of the parts list
- TP6: value TestPoint -> EPD_SW_TP; now left out of the parts list
- U1: value STM32G030K6Tx -> STM32G031K6Tx; symbol MCU_ST_STM32G0:STM32G030K6Tx -> MCU_ST_STM32G0:STM32G031K6Tx; JLCPCB C529331 -> C432202; LCSC (none) -> C432202; MPN (none) -> STM32G031K6T6
- U2: value ST25DV64K-IER8S3 -> ST25DV64KC-IE8C3; symbol RF_NFC:ST25DV04K-IER8C3 -> RF_NFC:ST25DV64K-IER8C3; JLCPCB C1852798 -> C5267462; LCSC (none) -> C5267462; MPN (none) -> ST25DV64KC-IE8C3
- U3: JLCPCB (none) -> C2681320; LCSC (none) -> C2681320; MPN (none) -> TPS22917DBVR
Connections:
- net EPD_SW: now also R14.2
- net GND: now also J1.17 (Pin_17), C28.2, C29.2, C30.2, C31.2, C32.2, C39.2, C40.2, C41.2, C42.2, C43.2, C44.2, C45.2, C46.2, C47.2, C48.2, C49.2, J3.2 (Pin_2), R10.2, R11.2, R7.2, R9.2, U4.2 (GND), U5.1 (GND), U6.2 (GND), U6.3 (~{CE}), U7.11 (GND), U7.2 (SEL), U7.8 (GND); no longer C19.2, J1.20 (Pin_20)
- net NFC_INT: now also R13.1
- net SYS_VDD: now also C19.2, C47.1, R13.2, R8.1, TP8.1, U4.6 (VOUT); no longer C14.1, C15.1, C16.1, C17.1, C25.1, C26.1, D4.1 (K), TP1.1
- net V_EH_RAW: now also U6.1 (VIN)
- net U3_CT: now reaches C19.1, U3.4 (CT)
- net PWR_HOLD: now reaches R3.2, R5.1, U1.7 (PA0)
- net PWR_HOLD: now also D6.2 (A)
- net at C2.1: now also J1.20 (Pin_20); no longer J1.17 (Pin_17)
- net at U3.5 (QOD): now also R14.1
- new net CFG1: R9.1, U7.3 (CFG1)
- new net CFG2: R10.1, U7.4 (CFG2)
- new net CFG3: R11.1, U7.5 (CFG3)
- new net EN_3V3: R12.2, TP12.1, U7.1 (EN)
- new net LX1: L2.1, U7.9 (LX1)
- new net LX2: L2.2, U7.7 (LX2)
- new net PWR_GOOD: D5.2 (A), U5.2 (~{RESET})
- new net PWR_REQ: D5.1 (K), D6.1 (K), R7.1, TP9.1, U4.3 (ON)
- new net U4_CT: C27.1, U4.4 (CT)
- new net U4_QOD: R8.2, U4.5 (QOD)
- new net VRAW: C25.1, C26.1, C39.1, C40.1, C41.1, D4.1 (K), R12.1, TP10.1, U6.6 (VOUT), U7.10 (VIN)
- new net VRES_3V3: C14.1, C15.1, C16.1, C17.1, C27.2, C28.1, C29.1, C30.1, C31.1, C32.1, C42.1, C43.1, C44.1, C45.1, C46.1, C48.1, C49.1, J3.1 (Pin_1), TP1.1, TP11.1, U4.1 (VIN), U5.3 (VDD), U7.6 (VOUT)
- no-connect marks 18 -> 22
Other:
- note added: "C19/C27 are CT-to-VIN (never CT-to-GND). Model the PCB coil as a 2-terminal inductor/net-tie before adding tuning C; keep copper away above/below the antenna."
- note added: "POWER PARTS: U6 LM66100 active, D4 DNP fallback; U7 TPS63900=3.3V/2.5mA; VRES nominal 1.6504mF (7x220uF + 5x22uF + 4x100nF). Validate leakage, charge time and min VDD."
- note added: "POWER: U5 (2.93V) + PWR_HOLD -> D5/D6 -> PWR_REQ -> U4 ON. STM32G031 BOR3/PVD4 handle undervoltage; release PWR_HOLD only after EPD OFF."
- note added: "U2 ST25DV64KC-IE8C3: provision EH_MODE=0; stage image+CRC in EEPROM; stop RF traffic while TPS63900 charges VRES_3V3."
- note added: "VERIFY BEFORE ORDER: VRAW stays >=1.8V while charging; VRES_3V3 reaches 3.20V; SYS_VDD stays >=2.80V during full-screen Partial."
- moved on the sheet: C2

Commit message: implement few adjustment on footprints/circuit, update readme
Parts:
- U1: value STM32G031K6Tx -> STM32G031K8T6; symbol MCU_ST_STM32G0:STM32G031K6Tx -> MCU_ST_STM32G0:STM32G031K8Tx; JLCPCB C432202 -> C432203; LCSC C432202 -> C432203; MPN STM32G031K6T6 -> STM32G031K8T6
- U2: value ST25DV64KC-IE8C3 -> ST25DV04K-IER6C3; symbol RF_NFC:ST25DV64K-IER8C3 -> RF_NFC:ST25DV04K-IER8C3; JLCPCB C5267462 -> C2908287; LCSC C5267462 -> C2908287; MPN ST25DV64KC-IE8C3 -> ST25DV04K-IER6C3
Other:
- note added: "U2 ST25DV04K-IER6C3: provision EH_MODE=0, FTM.MB_MODE=1; use the 256-byte FTM mailbox; images live in MCU Flash; pause RF traffic while VRES_3V3 charges."
- note removed: "U2 ST25DV64KC-IE8C3: provision EH_MODE=0; stage image+CRC in EEPROM; stop RF traffic while TPS63900 charges VRES_3V3."
Changed lines of the file:
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@@
 		)
 	)
-	(text "U2 ST25DV64KC-IE8C3: provision EH_MODE=0; stage image+CRC in EEPROM; stop RF traffic while TPS63900 charges VRES_3V3."
+	(text "U2 ST25DV04K-IER6C3: provision EH_MODE=0, FTM.MB_MODE=1; use the 256-byte FTM mailbox; images live in MCU Flash; pause RF traffic while VRES_3V3 charges."
 		(exclude_from_sim no)
 		(at 100 194 0)
@@
 	)
 	(symbol
-		(lib_id "RF_NFC:ST25DV64K-IER8C3")
+		(lib_id "RF_NFC:ST25DV04K-IER8C3")
 		(at 125.73 133.35 0)
 		(unit 1)
@@
 			)
 		)
-		(property "Value" "ST25DV64KC-IE8C3"
+		(property "Value" "ST25DV04K-IER6C3"
 			(at 136.525 139.7 0)
 			(show_name no)
@@
 			)
 		)
-		(property "Datasheet" "https://www.st.com/resource/en/datasheet/st25dv64kc.pdf"
+		(property "Datasheet" "https://www.st.com/resource/en/datasheet/st25dv04k.pdf"
 			(at 125.73 133.35 0)
 			(hide yes)
@@
 			)
 		)
-		(property "Description" "64-Kbit dynamic NFC/RFID tag with 8192-byte EEPROM, 256-byte mailbox and energy harvesting, UFDFPN-8"
+		(property "Description" "4-Kbit dynamic NFC/RFID tag with 512-byte EEPROM, 256-byte mailbox and energy harvesting, UFDFPN-8"
 			(at 125.73 133.35 0)
 			(hide yes)
@@
 			)
 		)
-		(property "JLCPCB" "C5267462"
+		(property "JLCPCB" "C2908287"
 			(at 125.73 133.35 0)
 			(hide yes)
@@
 			)
 		)
-		(property "LCSC" "C5267462"
+		(property "LCSC" "C2908287"
 			(at 125.73 133.35 0)
 			(hide yes)
@@
 			)
 		)
-		(property "MPN" "ST25DV64KC-IE8C3"
+		(property "MPN" "ST25DV04K-IER6C3"
 			(at 125.73 133.35 0)
 			(hide yes)
@@
 	)
 	(symbol
-		(lib_id "MCU_ST_STM32G0:STM32G031K6Tx")
+		(lib_id "MCU_ST_STM32G0:STM32G031K8Tx")
 		(at 44.45 115.57 0)
 		(unit 1)
@@
 			)
 		)
-		(property "Value" "STM32G031K6Tx"
+		(property "Value" "STM32G031K8T6"
 			(at 46.5933 87.63 0)
 			(show_name no)
@@
 			)
 		)
-		(property "Datasheet" "https://www.st.com/resource/en/datasheet/stm32g031k6.pdf"
+		(property "Datasheet" "https://www.st.com/resource/en/datasheet/stm32g031k8.pdf"
 			(at 44.45 115.57 0)
 			(hide yes)
@@
 			)
 		)
-		(property "Description" "STMicroelectronics Arm Cortex-M0+ MCU, 32KB flash, 8KB RAM, 64 MHz, 1.7-3.6V, 30 GPIO, LQFP32"
+		(property "Description" "STMicroelectronics Arm Cortex-M0+ MCU, 64KB flash, 8KB RAM, 64 MHz, 1.7-3.6V, 30 GPIO, LQFP32"
 			(at 44.45 115.57 0)
 			(hide yes)
@@
 			)
 		)
-		(property "MPN" "STM32G031K6T6"
+		(property "MPN" "STM32G031K8T6"
 			(at 44.45 115.57 0)
 			(hide yes)
@@
 			)
 		)
-		(property "LCSC" "C432202"
+		(property "LCSC" "C432203"
 			(at 44.45 115.57 0)
 			(hide yes)
@@
 			)
 		)
-		(property "JLCPCB" "C432202"
+		(property "JLCPCB" "C432203"
 			(at 44.45 115.57 0)
 			(hide yes)

Commit message: feat: Add production files for Maker Faire Tokyo 2026, including BOM, CPL, and Gerber data
Parts:
- L1: JLCPCB C6364799 -> C167813; LCSC C6364799 -> C167813; MPN ANR4020T470M -> FNR4018S470MT
Changed lines of the file:
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@@
 			)
 		)
-		(property "Datasheet" "https://datasheet.lcsc.com/datasheet/pdf/bb7b99ff1be8bff44e9ef21ee7214f91.pdf?productCode=C6364799"
+		(property "Datasheet" "https://jlcpcb.com/partdetail/179196-FNR4018S470MT/C167813"
 			(at 127 74.93 0)
 			(hide yes)
@@
 			)
 		)
-		(property "Description" "47uH 610mA Irms 810mA Isat shielded power inductor, 4x4x2mm"
+		(property "Description" "47uH 650mA rated 700mA saturation 845mOhm shielded power inductor, SMD 4x4mm"
 			(at 127 74.93 0)
 			(hide yes)
@@
 			)
 		)
-		(property "JLCPCB" "C6364799"
+		(property "JLCPCB" "C167813"
 			(at 127 74.93 0)
 			(hide yes)
@@
 			)
 		)
-		(property "LCSC" "C6364799"
+		(property "LCSC" "C167813"
 			(at 127 74.93 0)
 			(hide yes)
@@
 			)
 		)
-		(property "MPN" "ANR4020T470M"
+		(property "MPN" "FNR4018S470MT"
 			(at 127 74.93 0)
 			(hide yes)
