File: namecard.kicad_pcb (KiCad board)
At the start: 2 copper layers, 85.6 x 54 mm, 43 parts, among them J1 Conn_01x24, J2 Conn_01x05, Q1 AO3400A, U1 STM32G030K6Tx, U2 ST25DV04K-IER8C3, U3 TPS22917DBV

Commit message: wip: 配置を更新
Parts:
- added C20: 100nf, Capacitor_SMD:C_0603_1608Metric, F.Cu at (128.5, 97.0)
- added C24: 0.1uf, Capacitor_SMD:C_0805_2012Metric, F.Cu at (135.0, 84.0)
- added C25: 1uf, Capacitor_SMD:C_0805_2012Metric, F.Cu at (125.0, 92.5)
- added C26: 0.1uf, Capacitor_SMD:C_0805_2012Metric, F.Cu at (125.0, 90.5)
- C23: value 22uf -> 1uf
- moved TP7 5.41 mm to (122.0, 97.0)
- moved C14 4.92 mm to (121.0, 86.5), turned to 90 degrees
- moved C16 3.50 mm to (128.0, 86.5)
- moved C17 3.50 mm to (131.5, 86.5)
- moved C3 3.50 mm to (128.5, 100.5)
- moved C15 1.58 mm to (124.5, 86.5), turned to 90 degrees
- moved C19 0.50 mm to (117.5, 87.0)
- moved U3 0.50 mm to (117.5, 90.0)
Routing:
- net /SYS_VDD: track 77.4 -> 85.7 mm
- net /V_EH_RAW: track 16.0 -> 18.6 mm
- net Net-(D3-A): track 24.3 -> 25.5 mm
- net GND: track 19.8 -> 19.1 mm, vias 11 -> 12
- net /EPD_SW: track 72.5 -> 72.0 mm

Commit message: v4
Parts:
- added C27: 1nF, Capacitor_SMD:C_0402_1005Metric, F.Cu at (138.5, 93.5)
- added C28: 100nF, Capacitor_SMD:C_0402_1005Metric, F.Cu at (126.2, 92.5)
- added C29: 22uF 6.3V X5R, Capacitor_SMD:C_0805_2012Metric, F.Cu at (124.8, 93.2)
- added C30: 22uF 6.3V X5R, Capacitor_SMD:C_0805_2012Metric, F.Cu at (118.8, 97.5)
- added C31: 22uF 6.3V X5R, Capacitor_SMD:C_0805_2012Metric, F.Cu at (120.8, 97.5)
- added C32: 22uF 6.3V X5R, Capacitor_SMD:C_0805_2012Metric, F.Cu at (116.8, 97.5)
- added C39: 220uF/6.3V VRAW, Capacitor_Tantalum_SMD:CP_EIA-3528-21_Kemet-B, F.Cu at (140.5, 89.0)
- added C40: 10uF 25V X5R, Capacitor_SMD:C_0805_2012Metric, F.Cu at (135.5, 89.0)
- added C41: 100nF, Capacitor_SMD:C_0402_1005Metric, F.Cu at (137.2, 85.5)
- added C42: 22uF 6.3V X5R, Capacitor_SMD:C_0805_2012Metric, F.Cu at (132.0, 89.0)
- added C43: 100nF, Capacitor_SMD:C_0402_1005Metric, F.Cu at (133.8, 88.2)
- added C44: 100nF, Capacitor_SMD:C_0402_1005Metric, F.Cu at (128.8, 88.7)
- added C45: 100nF, Capacitor_SMD:C_0402_1005Metric, F.Cu at (139.5, 92.5)
- added C46: 220uF/6.3V VRES, Capacitor_Tantalum_SMD:CP_EIA-3528-21_Kemet-B, F.Cu at (112.5, 93.0)
- added C47: 100nF U2 DECOUPLING, Capacitor_SMD:C_0603_1608Metric, F.Cu at (144.5, 78.5)
- added C48: 220uF/6.3V VRES, Capacitor_Tantalum_SMD:CP_EIA-3528-21_Kemet-B, F.Cu at (116.2, 93.0)
- added C49: 220uF/6.3V VRES, Capacitor_Tantalum_SMD:CP_EIA-3528-21_Kemet-B, F.Cu at (120.0, 93.0)
- added D5: 1N4148W, Diode_SMD:D_SOD-123, F.Cu at (129.2, 95.8)
- added D6: 1N4148W, Diode_SMD:D_SOD-123, F.Cu at (134.2, 95.8)
- added J3: EXT_VRES_CAP_DNP, Connector_PinHeader_2.54mm:PinHeader_1x02_P2.54mm_Vertical, F.Cu at (113.2, 82.0)
- added L2: 2.2uH, Inductor_SMD:L_Sunlord_SWPA252012S, F.Cu at (135.2, 84.9)
- added R10: 5.11k 1% (2.5mA), Resistor_SMD:R_0402_1005Metric, F.Cu at (128.2, 85.4)
- added R11: 16.2k 1%, Resistor_SMD:R_0402_1005Metric, F.Cu at (128.2, 86.4)
- added R12: 0R, Resistor_SMD:R_0402_1005Metric, F.Cu at (131.5, 82.9)
- added R13: 10k GPO PULLUP, Resistor_SMD:R_0603_1608Metric, F.Cu at (146.2, 81.5)
- added R14: 1k EPD DISCHARGE, Resistor_SMD:R_0603_1608Metric, F.Cu at (139.0, 98.5)
- added R7: 4.7M, Resistor_SMD:R_0402_1005Metric, F.Cu at (131.0, 98.0)
- added R8: 1k, Resistor_SMD:R_0402_1005Metric, F.Cu at (137.5, 92.5)
- added R9: 36.5k 1%, Resistor_SMD:R_0402_1005Metric, F.Cu at (128.2, 84.4)
- added TP10: VRAW_TP, TestPoint:TestPoint_Pad_D1.0mm, F.Cu at (130.8, 80.0)
- added TP11: VRES_3V3_TP, TestPoint:TestPoint_Pad_D1.0mm, F.Cu at (109.2, 90.2)
- added TP12: EN_3V3_TP, TestPoint:TestPoint_Pad_D1.0mm, F.Cu at (127.8, 80.0)
- added TP8: SYS_VDD_TP, TestPoint:TestPoint_Pad_D1.0mm, F.Cu at (124.0, 101.0)
- added TP9: PWR_REQ_TP, TestPoint:TestPoint_Pad_D1.0mm, F.Cu at (120.5, 101.0)
- added U4: TPS22917DBV, Package_TO_SOT_SMD:SOT-23-6, F.Cu at (134.2, 92.5)
- added U5: TPS3839K33DBZR, Package_TO_SOT_SMD:SOT-23, F.Cu at (128.8, 92.5)
- added U6: LM66100, Package_TO_SOT_SMD:SOT-363_SC-70-6, F.Cu at (138.2, 82.5)
- added U7: TPS63900, Package_SON:WSON-10-1EP_2.5x2.5mm_P0.5mm_EP1.2x2mm_ThermalVias, F.Cu at (131.5, 84.9)
- C1, C10, C11, C12, C2, C5, C6, C7, C9: value 1uF -> 1uF 50V X5R
- C14, C15, C16, C17: value 220uf -> 220uF/6.3V; footprint Capacitor_Tantalum_SMD:6TPE220MAZB -> Capacitor_Tantalum_SMD:CP_EIA-3528-21_Kemet-B
- C19: value 1nf -> 1nF
- C3: value 4.7uF -> 4.7uF 25V X5R; footprint Capacitor_SMD:C_0603_1608Metric -> Capacitor_SMD:C_0805_2012Metric
- C4: value 4.7uF -> 4.7uF 16V X5R
- D1, D2, D3: value MBR0530 -> MBR0530T1G
- D4: value D_Schottky -> DNP SCHOTTKY
- L1: footprint Inductor_SMD:L_1210_3225Metric -> Inductor_SMD:L_APV_ANR4020
- R3: value 1M -> 1M DNP
- R5: value 470k -> 470k DNP
- TP1: value TestPoint -> VRES_3V3_TP
- TP3: value TestPoint -> V_EH_RAW_TP
- TP6: value TestPoint -> EPD_SW_TP
- U1: value STM32G030K6Tx -> STM32G031K6Tx
- U2: value ST25DV04K-IER8C3 -> ST25DV64KC-IE8C3
- moved R2 34.0 mm to (151.4, 99.2)
- moved R1 33.9 mm to (151.4, 100.8)
- moved Q1 33.9 mm to (147.4, 98.8)
- moved L1 30.6 mm to (142.5, 102.0), turned to 180 degrees
- moved U3 26.8 mm to (143.1, 97.8), turned to 180 degrees
- moved C5 26.6 mm to (151.4, 102.2), turned to 180 degrees
- moved D3 26.0 mm to (147.4, 101.8)
- moved C19 23.7 mm to (139.0, 97.0)
- moved C4 23.0 mm to (139.2, 101.5), turned to -90 degrees
- moved TP6 19.8 mm to (127.5, 101.0)
- moved C20 14.9 mm to (142.8, 92.5), turned to -90 degrees
- moved TP3 13.5 mm to (149.2, 80.5)
- moved TP1 13.2 mm to (120.0, 80.0)
- moved R3 13.2 mm to (146.0, 92.2)
- moved C18 11.5 mm to (158.3, 99.0), turned to 0 degrees
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Connections:
- net Net-(U1-PA0) renamed /PWR_HOLD
- net Net-(U3-CT) renamed /U3_CT
- C14 pad 1: /SYS_VDD -> /VRES_3V3
- C15 pad 1: /SYS_VDD -> /VRES_3V3
- C16 pad 1: /SYS_VDD -> /VRES_3V3
- C17 pad 1: /SYS_VDD -> /VRES_3V3
- C19 pad 2: GND -> /SYS_VDD
- C2 pad 1: Net-(J1-Pin_17) -> Net-(J1-Pin_20)
- C25 pad 1: /SYS_VDD -> /VRAW
- C26 pad 1: /SYS_VDD -> /VRAW
- D4 pad 1: /SYS_VDD -> /VRAW
- J1 pad 17: Net-(J1-Pin_17) -> GND
- J1 pad 20: GND -> Net-(J1-Pin_20)
- TP1 pad 1: /SYS_VDD -> /VRES_3V3
- U3 pad 5: unconnected-(U3-QOD-Pad5) -> Net-(U3-QOD)
Routing:
- net /VRES_3V3: track 0.00 -> 98.0 mm, vias 0 -> 4
- net /RESE: track 57.3 -> 20.5 mm
- net /GDR: track 58.4 -> 22.2 mm
- net Net-(U2-AC0): track 1261.6 -> 1227.4 mm, vias 4 -> 2
- net /VRAW: track 0.00 -> 32.3 mm, vias 0 -> 2
- net GND: track 19.1 -> 47.0 mm, vias 12 -> 11
- net /PREVGH: track 44.4 -> 17.6 mm
- net /EPD_SW: track 72.0 -> 49.8 mm
- net /PWR_REQ: track 0.00 -> 19.4 mm
- net Net-(U1-PA6): track 30.9 -> 11.8 mm
- net /NRST: track 31.7 -> 16.6 mm
- net /NFC_INT: track 16.0 -> 30.0 mm, vias 2 -> 3
- net /SPI_MOSI: track 27.3 -> 13.6 mm
- net Net-(D3-A): track 25.5 -> 12.0 mm, vias 0 -> 2
- net Net-(J1-Pin_7): track 15.3 -> 1.92 mm, vias 2 -> 0
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Other:
- board text added: "TP3"

Commit message: V5: release firmware, hardware, software
Parts:
- removed TP11: VRES_3V3_TP, TestPoint:TestPoint_Pad_D1.0mm
- added REF**: MountingHole_2.2mm_M2, MountingHole:MountingHole_2.2mm_M2, F.Cu at (101.8, 74.5)
- added REF**: MountingHole_2.2mm_M2, MountingHole:MountingHole_2.2mm_M2, F.Cu at (168.8, 74.5)
- added REF**: MountingHole_2.2mm_M2, MountingHole:MountingHole_2.2mm_M2, F.Cu at (168.8, 111.5)
- added REF**: MountingHole_2.2mm_M2, MountingHole:MountingHole_2.2mm_M2, F.Cu at (101.8, 111.5)
- 3V3 EN: renamed from TP12
- EPD PWR: renamed from TP6
- EXT CAP: renamed from J3
- PWR REQ: renamed from TP9
- SYS 3V3: renamed from TP8
- moved U2 4.38 mm to (146.5, 74.2)
- moved C47 2.76 mm to (147.2, 78.8)
- renumbered TP7 to GND, TP5 to GPIO1, TP4 to GPIO2, TP10 to VRAW
Routing:
- net /VRES_3V3: track 98.0 -> 85.9 mm
- net /SYS_VDD: track 80.9 -> 74.1 mm
- net GND: track 47.0 -> 51.4 mm
- net /NFC_INT: track 30.0 -> 28.0 mm, vias 3 -> 2
- net /I2C_SCL: track 17.4 -> 16.2 mm
- net /I2C_SDA: track 17.8 -> 17.3 mm
Other:
- outline, holes or cut-outs redrawn
- board text added: "EH_RAW"
- board text added: "VSTORE"
- board text removed: "TP3"

Commit message: implement few adjustment on footprints/circuit, update readme
Parts:
- U1: value STM32G031K6Tx -> STM32G031K8T6
- U2: value ST25DV64KC-IE8C3 -> ST25DV04K-IER6C3
Changed lines of the file:
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@@
 			)
 		)
-		(property "Value" "ST25DV64KC-IE8C3"
+		(property "Value" "ST25DV04K-IER6C3"
 			(at 0 2.05 90)
 			(layer "F.Fab")
@@
 			)
 		)
-		(property "JLCPCB" "C5267462"
-			(at 0 0 270)
-			(unlocked yes)
-			(layer "F.Fab")
-			(hide yes)
-			(effects
-				(font
-					(size 1 1)
-					(thickness 0.15)
-				)
-			)
-		)
-		(property "LCSC" "C5267462"
-			(at 0 0 270)
-			(unlocked yes)
-			(layer "F.Fab")
-			(hide yes)
-			(effects
-				(font
-					(size 1 1)
-					(thickness 0.15)
-				)
-			)
-		)
-		(property "MPN" "ST25DV64KC-IE8C3"
+		(property "JLCPCB" "C2908287"
+			(at 0 0 270)
+			(unlocked yes)
+			(layer "F.Fab")
+			(hide yes)
+			(effects
+				(font
+					(size 1 1)
+					(thickness 0.15)
+				)
+			)
+		)
+		(property "LCSC" "C2908287"
+			(at 0 0 270)
+			(unlocked yes)
+			(layer "F.Fab")
+			(hide yes)
+			(effects
+				(font
+					(size 1 1)
+					(thickness 0.15)
+				)
+			)
+		)
+		(property "MPN" "ST25DV04K-IER6C3"
 			(at 0 0 270)
 			(unlocked yes)
@@
 			)
 		)
-		(property "Value" "STM32G031K6Tx"
+		(property "Value" "STM32G031K8T6"
 			(at 0 5.88 0)
 			(layer "F.Fab")
@@
 			)
 		)
-		(property "JLCPCB" "C432202"
-			(at 0 0 0)
-			(unlocked yes)
-			(layer "F.Fab")
-			(hide yes)
-			(effects
-				(font
-					(size 1 1)
-					(thickness 0.15)
-				)
-			)
-		)
-		(property "MPN" "STM32G031K6T6"
-			(at 0 0 0)
-			(unlocked yes)
-			(layer "F.Fab")
-			(hide yes)
-			(effects
-				(font
-					(size 1 1)
-					(thickness 0.15)
-				)
-			)
-		)
-		(property "LCSC" "C432202"
-			(at 0 0 0)
-			(unlocked yes)
+		(property "JLCPCB" "C432203"
+			(at 0 0 0)
+			(unlocked yes)
+			(layer "F.Fab")
+			(hide yes)
+			(effects
+				(font
+					(size 1 1)
+					(thickness 0.15)
+				)
+			)
+		)
+		(property "MPN" "STM32G031K8T6"
+			(at 0 0 0)
+			(unlocked yes)
+			(layer "F.Fab")
+			(hide yes)
+			(effects
+				(font
+					(size 1 1)
+					(thickness 0.15)
+				)
+			)
+		)
+		(property "LCSC" "C432203"
+			(at 0 0 0)
+			(unlocked yes)
